File: RGBW_board.sch (KiCad schematic (older format))
At the start: 13 parts, among them J1 Jack-DC, J2 Conn_01x02, J3 Conn_01x04, J4 Conn_01x02, Q1 2N7002, Q2 2N7002, Q3 2N7002, Q4 2N7002, U1 WeMos_mini

Commit message: --REV1-- Added rev1 to project git
Parts:
- removed J1: Jack-DC, Connectors:BARREL_JACK, symbol Jack-DC
- removed J2: Conn_01x02, Pin_Headers:Pin_Header_Angled_1x02_Pitch2.54mm, symbol Conn_01x02
- removed Q1, Q2, Q3, Q4: 2N7002, TO_SOT_Packages_SMD:SOT-23, symbol 2N7002-RESCUE-RGBW_board
- added C1, C2, C3, C4: C_Small, Capacitors_SMD:C_1210, symbol C_Small
- added J1: BTNs, Connectors_Molex:Molex_KK-6410-03_03x2.54mm_Straight, symbol Conn_01x03
- added J5: Jack-DC, Connectors:BARREL_JACK, symbol Jack-DC
- added Q1, Q2, Q3, Q4: 2N7002, TO_SOT_Packages_SMD:SOT-23, symbol 2N7002
- added U2, U3: Mini_DC-DC_4.5-24V_to_0.8-17V, kenneth:Mini_DC-DC_converter, symbol Mini_DC-DC_4.5-24V_to_0.8-17V
- J3: value Conn_01x04 -> RGB; footprint Pin_Headers:Pin_Header_Angled_1x04_Pitch2.54mm -> Connectors_Molex:Molex_KK-6410-04_04x2.54mm_Straight
- J4: value Conn_01x02 -> White; footprint Pin_Headers:Pin_Header_Angled_1x02_Pitch2.54mm -> Connectors_Molex:Molex_KK-6410-02_02x2.54mm_Straight
Connections:
- net labels added: +24V, 5V, BTN0, BTN1, Enable
- wire segments 47 -> 77
- no-connect marks 0 -> 8

Commit message: --REV2-- Added rev2 to git project
Parts:
- added J2: Conn_01x02, kenneth:Battery_wirePad_SMD, symbol Conn_01x02
- added JP1: Jumper_NC_Dual, kenneth:Jumper_dual, symbol Jumper_NC_Dual
- added JP2: Jumper_NO_Small, Resistors_SMD:R_0805, symbol Jumper_NO_Small
- U2, U3: footprint kenneth:Mini_DC-DC_converter -> kenneth:Mini_DC-DC_converter_RED
Connections:
- net labels added: 5Vor3V3
- net labels removed: 5V, Enable
- wire segments 77 -> 90
- no-connect marks 8 -> 9
Changed lines of the file:
@@
 F 0 "U2" H 9950 4800 60  0000 C CNN
 F 1 "Mini_DC-DC_4.5-24V_to_0.8-17V" H 9650 4200 60  0001 C CNN
-F 2 "kenneth:Mini_DC-DC_converter" H 9150 4350 60  0001 C CNN
+F 2 "kenneth:Mini_DC-DC_converter_RED" H 9150 4350 60  0001 C CNN
 F 3 "" H 9150 4350 60  0001 C CNN
 	1    9150 4350
@@
 F 0 "U3" H 9950 6050 60  0000 C CNN
 F 1 "Mini_DC-DC_4.5-24V_to_0.8-17V" H 9650 5450 60  0001 C CNN
-F 2 "kenneth:Mini_DC-DC_converter" H 9150 5600 60  0001 C CNN
+F 2 "kenneth:Mini_DC-DC_converter_RED" H 9150 5600 60  0001 C CNN
 F 3 "" H 9150 5600 60  0001 C CNN
 	1    9150 5600
@@
 	1    0    0    -1
 $EndComp
-Text Label 8650 5300 0    60   ~ 0
-Enable
-Wire Wire Line
-	8650 5300 8950 5300
 Wire Wire Line
 	8450 5350 8450 5400
@@
 	1    0    0    -1
 $EndComp
-Text Label 8800 4350 0    60   ~ 0
-5V
-Text Label 5150 2400 0    60   ~ 0
-5V
+Text Label 8600 4350 0    60   ~ 0
+5Vor3V3
 Wire Wire Line
 	8950 4250 8450 4250
@@
 	8450 4250 8450 4300
 Wire Wire Line
-	8950 4350 8800 4350
+	8600 4350 8950 4350
 $Comp
 L GND #PWR020
@@
 L GND #PWR022
 U 1 1 5D6EF8F7
-P 4950 2550
-F 0 "#PWR022" H 4950 2300 50  0001 C CNN
-F 1 "GND" H 4950 2400 50  0000 C CNN
-F 2 "" H 4950 2550 50  0001 C CNN
-F 3 "" H 4950 2550 50  0001 C CNN
-	1    4950 2550
-	1    0    0    -1
-$EndComp
-Wire Wire Line
-	5300 2500 4950 2500
-Wire Wire Line
-	4950 2500 4950 2550
-Wire Wire Line
-	5300 2400 5150 2400
+P 4250 2600
+F 0 "#PWR022" H 4250 2350 50  0001 C CNN
+F 1 "GND" H 4250 2450 50  0000 C CNN
+F 2 "" H 4250 2600 50  0001 C CNN
+F 3 "" H 4250 2600 50  0001 C CNN
+	1    4250 2600
+	1    0    0    -1
+$EndComp
 Text Label 6550 2500 0    60   ~ 0
 RED_PWM_IN
-Text Label 6550 2600 0    60   ~ 0
+Text Label 6550 2900 0    60   ~ 0
 GREEN_PWM_IN
-Text Label 6550 2700 0    60   ~ 0
+Text Label 4600 2700 0    60   ~ 0
 BLUE_PWM_IN
-Text Label 6550 2800 0    60   ~ 0
+Text Label 4600 2600 0    60   ~ 0
 WHITE_PWM_IN
-Text Label 6550 2900 0    60   ~ 0
-Enable
 Wire Wire Line
 	6450 2500 7250 2500
 Wire Wire Line
-	6450 2600 7250 2600
-Wire Wire Line
-	6450 2700 7250 2700
-Wire Wire Line
-	6450 2800 7250 2800
-Wire Wire Line
 	6450 2900 7250 2900
-NoConn ~ 6450 2400
 NoConn ~ 6450 3000
 NoConn ~ 6450 3100
-NoConn ~ 5300 3100
-NoConn ~ 5300 3000
 NoConn ~ 5300 2900
 NoConn ~ 5300 2800
-Text Label 5100 2600 0    60   ~ 0
+Text Label 4600 3000 0    60   ~ 0
 BTN0
-Text Label 5100 2700 0    60   ~ 0
+Text Label 4600 3100 0    60   ~ 0
 BTN1
 Wire Wire Line
-	5100 2600 5300 2600
-Wire Wire Line
-	5100 2700 5300 2700
+	4600 2600 5300 2600
+Wire Wire Line
+	4600 2700 5300 2700
 Text Label 2600 6100 0    60   ~ 0
 BTN0
@@
 Wire Wire Line
 	2650 6200 2650 6250
+Text Label 6250 1750 2    60   ~ 0
+5Vor3V3
+$Comp
+L Jumper_NC_Dual JP1
+U 1 1 5D8227D8
+P 5850 2000
+F 0 "JP1" H 5900 1900 50  0000 L CNN
+F 1 "Jumper_NC_Dual" H 5850 2100 50  0001 C BNN
+F 2 "kenneth:Jumper_dual" H 5850 2000 50  0001 C CNN
+F 3 "" H 5850 2000 50  0001 C CNN
+	1    5850 2000
+	-1   0    0    1
+$EndComp
+Wire Wire Line
+	5850 1900 5850 1750
+Wire Wire Line
+	5850 1750 6250 1750
+Wire Wire Line
+	6100 2000 6550 2000
+Wire Wire Line
+	6550 2000 6550 2400
+Wire Wire Line
+	6550 2400 6450 2400
+Wire Wire Line
+	5600 2000 5200 2000
+Wire Wire Line
+	5200 2000 5200 2400
+Wire Wire Line
+	5200 2400 5300 2400
+NoConn ~ 6450 2600
+NoConn ~ 6450 2700
+NoConn ~ 6450 2800
+Wire Wire Line
+	5300 2500 4250 2500
+Wire Wire Line
+	4250 2500 4250 2600
+Wire Wire Line
+	5300 3000 4600 3000
+Wire Wire Line
+	5300 3100 4600 3100
+NoConn ~ 8950 5300
+$Comp
+L Conn_01x02 J2
+U 1 1 5D83A5F6
+P 10300 1300
+F 0 "J2" H 10300 1400 50  0000 C CNN
+F 1 "Conn_01x02" H 10300 1100 50  0000 C CNN
+F 2 "kenneth:Battery_wirePad_SMD" H 10300 1300 50  0001 C CNN
+F 3 "" H 10300 1300 50  0001 C CNN
+	1    10300 1300
+	-1   0    0    -1
+$EndComp
+$Comp
+L +24V #PWR024
+U 1 1 5D83A6EA
+P 10600 1250
+F 0 "#PWR024" H 10600 1100 50  0001 C CNN
+F 1 "+24V" H 10600 1390 50  0000 C CNN
+F 2 "" H 10600 1250 50  0001 C CNN
+F 3 "" H 10600 1250 50  0001 C CNN
+	1    10600 1250
+	1    0    0    -1
+$EndComp
+$Comp
+L GND #PWR025
+U 1 1 5D83A7AE
+P 10600 1550
+F 0 "#PWR025" H 10600 1300 50  0001 C CNN
+F 1 "GND" H 10600 1400 50  0000 C CNN
+F 2 "" H 10600 1550 50  0001 C CNN
+F 3 "" H 10600 1550 50  0001 C CNN
+	1    10600 1550
+	1    0    0    -1
+$EndComp
+Wire Wire Line
+	10500 1400 10600 1400
+Wire Wire Line
+	10600 1400 10600 1550
+Wire Wire Line
+	10500 1300 10600 1300
+Wire Wire Line
+	10600 1300 10600 1250
+$Comp
+L Jumper_NO_Small JP2
+U 1 1 5D83CBCD
+P 8650 2050
+F 0 "JP2" H 8650 2130 50  0000 C CNN
+F 1 "Jumper_NO_Small" H 8660 1990 50  0000 C CNN
+F 2 "Resistors_SMD:R_0805" H 8650 2050 50  0001 C CNN
+F 3 "" H 8650 2050 50  0001 C CNN
+	1    8650 2050
+	1    0    0    -1
+$EndComp
+$Comp
+L +24V #PWR026
+U 1 1 5D83CDB2
+P 8400 1950
+F 0 "#PWR026" H 8400 1800 50  0001 C CNN
+F 1 "+24V" H 8400 2090 50  0000 C CNN
+F 2 "" H 8400 1950 50  0001 C CNN
+F 3 "" H 8400 1950 50  0001 C CNN
+	1    8400 1950
+	1    0    0    -1
+$EndComp
+$Comp
+L +12V #PWR027
+U 1 1 5D83CDFF
+P 8900 1950
+F 0 "#PWR027" H 8900 1800 50  0001 C CNN
+F 1 "+12V" H 8900 2090 50  0000 C CNN
+F 2 "" H 8900 1950 50  0001 C CNN
+F 3 "" H 8900 1950 50  0001 C CNN
+	1    8900 1950
+	1    0    0    -1
+$EndComp
+Wire Wire Line
+	8400 1950 8400 2050
+Wire Wire Line
+	8400 2050 8550 2050
+Wire Wire Line
+	8750 2050 8900 2050
+Wire Wire Line
+	8900 2050 8900 1950
 $EndSCHEMATC
